Commit message: Created inertial tags in the URDF

File: src/my_robot_description/urdf/base_and_links.xacro (robot description, xacro)
@@ -1,5 +1,5 @@
 <?xml version="1.0"?>
 <robot xmlns:xacro = "http://www.ros.rog/wiki/xacro">
-        <xacro:property name = "base_length" value = "1"/>
+        <xacro:property name = "base_length" value = "0.5"/>
         <xacro:macro name = "wheel_link" params = 'prefix'>
             <link name = "${prefix}_wheel_link">
@@ -21,4 +21,6 @@
                     <material name="green"></material>
                 </visual>
+                <xacro:box_inertia m = "5.0" x = "0.6" y = "0.4" z = "0.2"
+                                    o_xyz = "0 0 0.1" o_rpy = "0 0 0"/>
             </link>
             <link name="caster_wheel">

File: src/my_robot_description/urdf/common_properties.xacro (robot description, xacro)
@@ -4,3 +4,12 @@
     <material name="somethingshit"><color rgba="0 0 0.8 1"></color></material>
     <material name="caster_wheel"><color rgba="1 0 0 1"></color></material>
+    <xacro:macro name = "box_inertia" params = "m x y z o_xyz o_rpy">
+        <inertial>
+                <mass value = "${m}"/>
+                <origin xyz = "${o_xyz}" rpy = "${o_rpy}"/>
+                <inertia ixx = "${(m / 12) * (y*y + z*z)}" ixy = "0" ixz = "0"
+                            iyy = "${(m / 12) * (x*x + z*z)}" iyz = "0"
+                            izz = "${(m / 12) * (x*x + y*y)}" />
+        </inertial>
+    </xacro:macro>
 </robot>

Commit message: Introduced collision boxes in the URDF.

File: src/my_robot_description/urdf/base_and_links.xacro (robot description, xacro)
@@ -11,5 +11,12 @@
                     <material name="somethingshit"></material>
                 </visual>
-                </link>
+                <collision>
+                    <geometry>
+                        <sphere radius = "0.1"></sphere>
+                    </geometry>
+                    <origin xyz="0 0 0" rpy="0 0 0"/>
+                </collision>
+                <xacro:wheel_inertia m = "0.2" r = "0.1" h = "0.05" o_xyz = "${-base_length / 4} 0.225 0" o_rpy = "${pi} 0 0"/>
+            </link>
         </xacro:macro>
         <link name="base_link">
@@ -21,4 +28,10 @@
                     <material name="green"></material>
                 </visual>
+                <collision>
+                    <geometry>
+                        <box size="${base_length} 0.4 0.2" />
+                    </geometry>
+                    <origin xyz="0 0 0.1" rpy="0 0 0" />
+                </collision>
                 <xacro:box_inertia m = "5.0" x = "0.6" y = "0.4" z = "0.2"
                                     o_xyz = "0 0 0.1" o_rpy = "0 0 0"/>
@@ -31,4 +44,13 @@
                     </geometry>
                 </visual>
+                <collision>
+                    <geometry>
+                        <sphere radius = "0.05"/>
+                        <material name="caster_wheel"/>
+                    </geometry>
+                    <origin xyz="0 0 0" rpy="0 0 0" />
+                </collision>
+                <xacro:castor_wheel_inertia m = "1.5" r = "0.05"
+                                    o_xyz = "0 0 -0.075" o_rpy = "0 0 0"/>
             </link>
             <xacro:wheel_link prefix = 'left'></xacro:wheel_link>

File: src/my_robot_description/urdf/common_properties.xacro (robot description, xacro)
@@ -13,3 +13,21 @@
         </inertial>
     </xacro:macro>
+    <xacro:macro name = "wheel_inertia" params = "m r h o_xyz o_rpy">
+        <inertial>
+                <mass value = "${m}"/>
+                <origin xyz = "${o_xyz}" rpy = "${o_rpy}"/>
+                <inertia ixx = "${(m / 12) * (3*r*r + h*h)}" ixy = "0" ixz = "0"
+                            iyy = "${(m / 12) * (3*r*r + h*h)}" iyz = "0"
+                            izz = "${0.5 * m * r * r}" />
+        </inertial>
+    </xacro:macro>
+    <xacro:macro name = "castor_wheel_inertia" params = "m r o_xyz o_rpy">
+        <inertial>
+                <mass value = "${m}"/>
+                <origin xyz = "${o_xyz}" rpy = "${o_rpy}"/>
+                <inertia ixx = "${(0.4 * m) * (r * r)}" ixy = "0" ixz = "0"
+                            iyy = "${(0.4 * m) * (r * r)}" iyz = "0"
+                            izz = "${(0.4 * m) * (r * r)}" />
+        </inertial>
+    </xacro:macro>
 </robot>
