Commit message: Successfully implemented a camera sensor and validated the video stream in RViz

File: src/my_robot_description/urdf/camera.xacro (robot description, xacro)
@@ -1,16 +1,21 @@
 <?xml version="1.0"?>
-<robot xmlns:xacro = "http://www.ros.rog/wiki/xacro">
-    <link name = "camera_link">
+<robot xmlns:xacro="http://www.ros.org/wiki/xacro">
+    <xacro:property name="camera_length" value="0.01" />
+    <xacro:property name="camera_width" value="0.1" />
+    <xacro:property name="camera_height" value="0.05" />
+    <link name="camera_link">
         <visual>
             <geometry>
-                <box size = "0.01 0.1 0.05"/>
+                <box size="${camera_length} ${camera_width} ${camera_height}" />
             </geometry>
+            <material name="grey" />
         </visual>
         <collision>
             <geometry>
-                <box size = "0.01 0.1 0.05"/>
+                <box size="${camera_length} ${camera_width} ${camera_height}" />
             </geometry>
         </collision>
-        <xacro:box_inertia m = "0.1" x = "0.01" y = "0.1" z = "0.05" o_xyz = "0 0 0" o_rpy = "0 0 0"/>
+        <xacro:box_inertia m="0.1" x="${camera_length}" y="${camera_width}" z="${camera_height}"
+                           o_xyz="0 0 0" o_rpy="0 0 0" />
     </link>
     <joint name = "base_camera_joint" type = "fixed">
@@ -19,3 +24,36 @@
         <origin xyz = "0.275 0 0.05" rpy = "0 0 0"/>
     </joint>
+    <link name="camera_link_optical" />
+    <joint name="camera_optical_joint" type="fixed">
+        <origin xyz="0 0 0" rpy="${-pi/2} 0 ${-pi/2}"/>
+        <parent link="camera_link"/>
+        <child link="camera_link_optical"/>
+    </joint>
+    <gazebo reference="camera_link">
+        <sensor name="camera" type="camera">
+            <camera>
+                <horizontal_fov>1.3962634</horizontal_fov>
+                <image>
+                    <width>640</width>
+                    <height>480</height>
+                    <format>R8G8B8</format>
+                </image>
+                <clip>
+                    <near>0.1</near>
+                    <far>15</far>
+                </clip>
+                <noise>
+                    <type>gaussian</type>
+                    <mean>0.0</mean>
+                    <stddev>0.007</stddev>
+                </noise>
+                <optical_frame_id>camera_link_optical</optical_frame_id>
+                <camera_info_topic>camera/camera_info</camera_info_topic>
+            </camera>
+            <always_on>1</always_on>
+            <update_rate>20</update_rate>
+            <visualize>true</visualize>
+            <topic>camera/image_raw</topic>
+        </sensor>
+    </gazebo>
 </robot>
