Commit message: Wrote a gazebo-ros bridge

File: src/my_robot_bringup/urdf/common_properties.xacro (robot description, xacro)
@@ -22,5 +22,5 @@
         </inertial>
     </xacro:macro>
-    <xacro:macro name = "castor_wheel_inertia" params = "m r o_xyz o_rpy">
+    <xacro:macro name = "caster_wheel_inertia" params = "m r o_xyz o_rpy">
         <inertial>
                 <mass value = "${m}"/>
